File: pcb/keyboard/v0.1/keyboard.kicad_sch (KiCad schematic)
At the start: 140 parts, among them SW1 A, SW10 A, SW11 A, SW12 A, SW13 A, SW14 A, SW15 A, SW16 A, SW17 A, SW18 A, SW19 A, SW2 A, SW20 A, SW21 A, SW22 A, SW23 A, SW24 A, SW25 A, SW26 A, SW27 A, SW28 A, SW29 A, SW3 A, SW30 A, SW31 A, SW32 A, SW33 A, SW34 A, SW35 A, SW36 A, SW37 A, SW38 A, SW39 A, SW4 A, SW40 A, SW41 A, SW42 A, SW43 A, SW44 A, SW45 A, SW46 A, SW47 A, SW48 A, SW49 A, SW5 A, SW50 A, SW51 A, SW52 A, SW53 A, SW54 A, SW55 A, SW56 A, SW57 A, SW58 A, SW59 A, SW6 A, SW60 A, SW61 A, SW62 A, SW63 A, SW7 A, SW8 A, SW9 A, U1 MDBT50Q-P1MV2, Y1 32.768

Commit message: Footprints for the two pogo pads
Parts:
- SW5: footprint (none) -> TH-A1OC:tact_switch_4.5x4.5_PTS647
Changed lines of the file:
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@@
 			)
 		)
-		(property "Footprint" ""
+		(property "Footprint" "TH-A1OC:tact_switch_4.5x4.5_PTS647"
 			(at 154.94 205.74 0)
 			(effects
