File: pcb/keyboard/v0.1/keyboard.kicad_sch (KiCad schematic)
At the start: 142 parts, among them J1 USB2.0, J2 SWD, SW1 BACKTICK, SW10 9, SW11 0, SW12 BACKSPACE, SW13 TAB, SW14 Q, SW15 W, SW16 E, SW17 R, SW18 T, SW19 Y, SW2 1, SW20 U, SW21 I, SW22 O, SW23 P, SW24 RETURN, SW25 CAPS, SW26 A, SW27 S, SW28 D, SW29 F, SW3 2, SW30 G, SW31 H, SW32 J, SW33 K, SW34 L, SW35 SEMI, SW36 QUOTE, SW37 LSHIFT, SW38 Z, SW39 X, SW4 3, SW40 C, SW41 V, SW42 B, SW43 N, SW44 M, SW45 COMMA, SW46 DOT, SW47 QUEST, SW48 RSHIFT, SW49 FN, SW5 4, SW50 LCTRL, SW51 LSUPER, SW52 LALT, SW53 SPACE, SW54 RALT, SW55 RSUPER, SW56 MENU, SW57 RCTRL, SW58 C1, SW59 C2, SW6 5, SW60 C3, SW61 C4, SW62 C5, SW63 C6, SW7 6, SW8 7, SW9 8, U1 MDBT50Q-P1MV2, Y1 32.768

Commit message: Rough layout
Connections:
- net VBUS: no longer J1.1 (VBUS), R1.1
- new net VBUS_USB: J1.1 (VBUS), R1.1
Changed lines of the file:
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@@
 		)
 	)
-	(label "VBUS"
+	(label "VBUS_USB"
 		(at 463.55 52.07 0)
 		(effects
