File: pcb/keyboard/v0.1/keyboard.kicad_pcb (KiCad board)
At the start: 2 copper layers, 80.9 x 104.7 mm, 142 parts, among them J1 USB2.0, J2 SWD, SW1 BACKTICK, SW10 9, SW11 0, SW12 BACKSPACE, SW13 TAB, SW14 Q, SW15 W, SW16 E, SW17 R, SW18 T, SW19 Y, SW2 1, SW20 U, SW21 I, SW22 O, SW23 P, SW24 RETURN, SW25 CAPS, SW26 A, SW27 S, SW28 D, SW29 F, SW3 2, SW30 G, SW31 H, SW32 J, SW33 K, SW34 L, SW35 SEMI, SW36 QUOTE, SW37 LSHIFT, SW38 Z, SW39 X, SW4 3, SW40 C, SW41 V, SW42 B, SW43 N, SW44 M, SW45 COMMA, SW46 DOT, SW47 QUEST, SW48 RSHIFT, SW49 FN, SW5 4, SW50 LCTRL, SW51 LSUPER, SW52 LALT, SW53 SPACE, SW54 RALT, SW55 RSUPER, SW56 MENU, SW57 RCTRL, SW58 C1, SW59 C2, SW6 5, SW60 C3, SW61 C4, SW62 C5, SW63 C6, SW7 6, SW8 7, SW9 8, U1 MDBT50Q-P1MV2, Y1 32.768

Commit message: Rough layout
Parts:
- moved TP1 115.0 mm to (43.4, 89.6)
- moved C1 95.3 mm to (76.7, 88.8)
- moved C2 94.9 mm to (77.6, 91.6), turned to 90 degrees
- moved JP1 92.1 mm to (67.6, 107.5), turned to 90 degrees
- moved TP2 91.9 mm to (80.4, 92.0)
- moved Y1 89.8 mm to (78.5, 98.5), turned to 180 degrees
- moved L1 87.4 mm to (75.7, 91.8), turned to -90 degrees
- moved D58 87.3 mm to (64.3, 111.4)
- moved D59 87.3 mm to (78.0, 111.4)
- moved D60 87.3 mm to (91.7, 111.4)
- moved D62 87.3 mm to (119.0, 111.4)
- moved D63 87.3 mm to (132.7, 111.4)
- moved D61 87.3 mm to (105.3, 111.4)
- moved SW58 87.3 mm to (59.8, 106.1)
- moved SW59 87.3 mm to (73.4, 106.1)
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Connections:
- J1 pad 1: /VBUS -> /VBUS_USB
- R1 pad 1: /VBUS -> /VBUS_USB
Other:
- board size 80.9 x 104.7 mm -> 80.8 x 79.7 mm
